Commit message: Satellite inertias

File: resources/robots/satellite/satellite.urdf (robot description, URDF)
Before this commit: robot satellite, 16 links, 15 joints
Links:
- added link arm_one, mass 0; visual cylinder length=0.5 radius=0.1
- added link arm_three, mass 10; visual cylinder length=2 radius=0.1
- added link arm_two, mass 10; visual cylinder length=2 radius=0.1
- link base_link: geometry visual box size=2.5 2.5 4
Joints:
- added joint arm_one_to_two: type revolute, parent arm_one, child arm_two, origin xyz=0 0 0, axis 0 1 0, limit lower=0 upper=3.14 effort=100.0 velocity=0.5
- added joint arm_two_to_three: type revolute, parent arm_two, child arm_three, origin xyz=0 0 2, axis 0 1 0, limit lower=-1.57 upper=1.57 effort=100.0 velocity=0.5
- added joint base_to_arm: type revolute, parent base_link, child arm_one, origin xyz=1.5 0 -0.25, axis 1 0 0, limit lower=-1.57 upper=1.57 effort=100.0 velocity=0.5

File: resources/robots/satellite/satellite.xacro (robot description, xacro)
@@ -17,4 +17,6 @@
     <xacro:property name="base_l" value="2" />
     <xacro:property name="base_h" value="4" />
+    <xacro:property name="arm_segment_length" value="2" />
+    <xacro:property name="arm_segment_mass" value="10" />
     <!-- <link name="base_dummy"></link> -->
     <!-- links -->
@@ -214,22 +216,55 @@
             <material name="white"/>
         </visual>
+        <inertial>
+            <mass value="0"/>
+            <origin xyz="0 0 0"/>
+            <inertia
+                ixx="0"
+                ixy="0.0" ixz="0.0"
+                iyy="0"
+                iyz="0.0"
+                izz="0"
+            />
+        </inertial>
     </link>
     <link name="arm_two">
         <visual>
             <geometry>
-                <cylinder length="2" radius="0.1"/>
+                <cylinder length="${arm_segment_length}" radius="0.1"/>
             </geometry>
             <origin rpy="0 0 0" xyz="0 0 1"/>
             <material name="white"/>
         </visual>
+        <inertial>
+            <mass value="${arm_segment_mass}"/>
+            <origin xyz="0 0 0"/>
+            <inertia
+                ixx="${1/3 * arm_segment_mass * arm_segment_length * arm_segment_length}"
+                ixy="0.0" ixz="0.0"
+                iyy="0"
+                iyz="0.0"
+                izz="${1/3 * arm_segment_mass * arm_segment_length * arm_segment_length}"
+            />
+        </inertial>
     </link>
     <link name="arm_three">
         <visual>
             <geometry>
-                <cylinder length="2" radius="0.1"/>
+                <cylinder length="${arm_segment_length}" radius="0.1"/>
             </geometry>
             <origin rpy="0 0 0" xyz="0.2 0 -1"/>
             <material name="white"/>
         </visual>
+        <inertial>
+            <mass value="${arm_segment_mass}"/>
+            <origin xyz="0 0 0"/>
+            <inertia
+                ixx="${1/3 * arm_segment_mass * arm_segment_length * arm_segment_length}"
+                ixy="0.0" ixz="0.0"
+                iyy="0"
+                iyz="0.0"
+                izz="${1/3 * arm_segment_mass * arm_segment_length * arm_segment_length}"
+            />
+        </inertial>
     </link>
     <joint name="base_to_arm" type="revolute">
