Commit message: New satellite models

File: resources/robots/satellite/satellite.motoman.urdf.xacro (robot description, xacro)
@@ -21,6 +21,6 @@
     <xacro:property name="base_l" value="4" />
     <xacro:property name="base_h" value="11" />
-    <xacro:property name="arm_segment_length" value="3" />
-    <xacro:property name="arm_segment_mass" value="136" />
+    <xacro:property name="arm_segment_length" value="2" />
+    <xacro:property name="arm_segment_mass" value="1" />
     <xacro:property name="show_outline" value="0" />
     <!-- <link name="base_dummy"></link> -->
@@ -33,7 +33,8 @@
         </inertial>
         <visual>
-            <origin rpy="0 0 1.57" xyz="0.1 0 -0.4"/>
-            <geometry>
-                <mesh filename="package://exotica_satellite_dynamics_solver/resources/robots/satellite/satellite_base2.dae" scale="1 1 1"/>
+            <origin rpy="0 0 0" xyz="0 0 0"/>
+            <geometry>
+                <!-- <mesh filename="package://exotica_satellite_dynamics_solver/resources/robots/satellite/satellite_base.dae" scale="1 1 1"/> -->
+          <mesh filename="package://ssl_1300_satellite_description/meshes/LORAL-1300MANIP.dae" />
             </geometry>
         </visual>
@@ -214,107 +215,10 @@
         <origin xyz="0 -1 -1"/>
     </joint>
-    <!-- arm -->
-    <link name="arm_base">
-        <visual>
-            <geometry>
-                <cylinder length="0.5" radius="0.1"/>
-            </geometry>
-            <origin rpy="0 0 0" xyz="0 0 0"/>
-            <material name="green"/>
-        </visual>
-        <inertial>
-            <mass value="1e-3"/>
-            <origin xyz="0 0 0"/>
-            <inertia ixx="1e-3" ixy="0.0" ixz="0.0" iyy="1e-3" iyz="0.0" izz="1e-3"/>
-        </inertial>
-    </link>
-    <link name="arm_shoulder">
-        <visual>
-            <geometry>
-                <cylinder length="${arm_segment_length}" radius="0.1"/>
-            </geometry>
-            <origin rpy="0 0 0" xyz="0 0 ${arm_segment_length/2}"/>
-            <material name="green"/>
-        </visual>
-        <inertial>
-            <mass value="${arm_segment_mass}"/>
-            <origin rpy="0 0 0" xyz="0 0 1"/>
-            <inertia ixx="${1/3 * arm_segment_mass * arm_segment_length * arm_segment_length}" ixy="0.0" ixz="0.0" iyy="1e-3" iyz="0.0" izz="${1/3 * arm_segment_mass * arm_segment_length * arm_segment_length}" />
-        </inertial>
-    </link>
-    <link name="arm_elbow">
-        <visual>
-            <geometry>
-                <cylinder length="${arm_segment_length}" radius="0.1"/>
-            </geometry>
-            <origin rpy="0 0 0" xyz="0.1 0 -${arm_segment_length/2}"/>
-            <material name="green"/>
-        </visual>
-        <inertial>
-            <mass value="${arm_segment_mass}"/>
-            <origin rpy="0 0 0" xyz="0 0 1"/>
-            <inertia ixx="${1/3 * arm_segment_mass * arm_segment_length * arm_segment_length}" ixy="0.0" ixz="0.0" iyy="1e-3" iyz="0.0" izz="${1/3 * arm_segment_mass * arm_segment_length * arm_segment_length}" />
-        </inertial>
-    </link>
-    <link name="arm_wrist">
-        <visual>
-            <geometry>
-                <cylinder length="${arm_segment_length}" radius="0.1"/>
-            </geometry>
-            <origin rpy="0 0 0" xyz="0.2 0 ${arm_segment_length/2}"/>
-            <material name="green"/>
-        </visual>
-        <inertial>
-            <mass value="${arm_segment_mass}"/>
-            <origin rpy="0 0 0" xyz="0 0 1"/>
-            <inertia ixx="${1/3 * arm_segment_mass * arm_segment_length * arm_segment_length}" ixy="0.0" ixz="0.0" iyy="1e-3" iyz="0.0" izz="${1/3 * arm_segment_mass * arm_segment_length * arm_segment_length}" />
-        </inertial>
-    </link>
-    <link name="arm_end_eff">
-        <visual>
-            <geometry>
-                <cylinder length="0.2" radius="0.1"/>
-            </geometry>
-            <origin rpy="0 0 0" xyz="0.2 0 0"/>
-            <material name="yellow"/>
-        </visual>
-        <inertial>
-            <mass value="1e-5"/>
-            <origin rpy="0 0 0" xyz="0 0 1"/>
-            <inertia ixx="1e-3" ixy="0.0" ixz="0.0" iyy="1e-3" iyz="0.0" izz="1e-3" />
-        </inertial>
-    </link>
-    <joint name="base_to_arm" type="revolute">
-        <parent link="base_link"/>
-        <child link="arm_base"/>
-        <limit effort="1.0" lower="-1.57" upper="1.57" velocity="0.5"/>
-        <axis xyz="1 0 0"/>
-        <origin xyz="1.25 0 -${arm_segment_length/2}"/>
-    </joint>
-    <joint name="arm_base_to_shoulder" type="revolute">
-        <parent link="arm_base"/>
-        <child link="arm_shoulder"/>
-        <limit effort="1.0" lower="0" upper="3.14" velocity="0.5"/>
-        <axis xyz="0 1 0"/>
-        <origin xyz="0 0 0"/>
-    </joint>
-    <joint name="arm_shoulder_to_elbow" type="revolute">
-        <parent link="arm_shoulder"/>
-        <child link="arm_elbow"/>
-        <limit effort="1.0" lower="0" upper="3.14" velocity="0.5"/>
-        <axis xyz="0 -1 0"/>
-        <origin xyz="0 0 ${arm_segment_length}"/>
-    </joint>
-    <joint name="arm_elbow_to_wrist" type="revolute">
-        <parent link="arm_elbow"/>
-        <child link="arm_wrist"/>
-        <limit effort="1.0" lower="-300" upper="300" velocity="0.5"/>
-        <axis xyz="-1 0 0"/>
-        <origin xyz="0 0 -${arm_segment_length}"/>
-    </joint>
-    <joint name="arm_wrist_to_end_eff" type="fixed">
-        <parent link="arm_wrist"/>
-        <child link="arm_end_eff"/>
-        <origin xyz="0 0 ${arm_segment_length + 0.1}"/>
+    <xacro:include filename="$(find ssl_1300_orbital_manipulator_description)/urdf/sia50_macro_with_approximate_inertia.xacro" />
+    <xacro:motoman_sia50 prefix="sia50d_"/>
+    <joint name="satellite_to_arm_joint" type="fixed">
+        <origin xyz="0 1.3 0" rpy="-1.57079632679 0 0"/>
+        <parent link="base_link"/>
+        <child link="sia50d_base_link"/>
     </joint>
 </robot>

File: resources/robots/satellite/satellite.noarm.urdf.xacro (robot description, xacro)
@@ -17,5 +17,5 @@
         <color rgba="1 1 1 1"/>
     </material>
-    <xacro:property name="base_mass" value="5190" />
+    <xacro:property name="base_mass" value="5000" />
     <xacro:property name="base_w" value="4" />
     <xacro:property name="base_l" value="4" />
@@ -23,5 +23,5 @@
     <xacro:property name="arm_segment_length" value="2" />
     <xacro:property name="arm_segment_mass" value="1" />
-    <xacro:property name="show_outline" value="1" />
+    <xacro:property name="show_outline" value="0" />
     <!-- <link name="base_dummy"></link> -->
     <!-- links -->
@@ -32,10 +32,11 @@
             <inertia ixx="${base_mass * 2.5 * 2.5 * 2/5}" ixy="0.0" ixz="0.0" iyy="${base_mass * 2.5 * 2.5 * 2/5}" iyz="0.0" izz="${base_mass * 4 * 4 * 2/5}" />
         </inertial>
-        <!-- <visual>
+        <visual>
             <origin rpy="0 0 0" xyz="0 0 0"/>
             <geometry>
-                <mesh filename="package://exotica_satellite_dynamics_solver/resources/robots/satellite/satellite_base.dae" scale="1 1 1"/>
-            </geometry>
-        </visual> -->
+                <!-- <mesh filename="package://exotica_satellite_dynamics_solver/resources/robots/satellite/satellite_base.dae" scale="1 1 1"/> -->
+          <mesh filename="package://ssl_1300_satellite_description/meshes/LORAL-1300MANIP.dae" />
+            </geometry>
+        </visual>
         <xacro:if value="${show_outline == 1}">
             <visual>

File: resources/robots/satellite/satellite.object.urdf.xacro (robot description, xacro)
@@ -17,5 +17,6 @@
         <color rgba="1 1 1 1"/>
     </material>
-    <xacro:property name="base_mass" value="5000" />
+    <xacro:property name="base_mass" value="11900" />
+    <xacro:property name="heavy_object_mass" value="100" />
     <xacro:property name="base_w" value="4" />
     <xacro:property name="base_l" value="4" />
@@ -23,5 +24,5 @@
     <xacro:property name="arm_segment_length" value="3" />
     <xacro:property name="arm_segment_mass" value="136" />
-    <xacro:property name="show_outline" value="0" />
+    <xacro:property name="show_outline" value="1" />
     <!-- <link name="base_dummy"></link> -->
     <!-- links -->
@@ -32,10 +33,10 @@
             <inertia ixx="${base_mass * 2.5 * 2.5 * 2/5}" ixy="0.0" ixz="0.0" iyy="${base_mass * 2.5 * 2.5 * 2/5}" iyz="0.0" izz="${base_mass * 4 * 4 * 2/5}" />
         </inertial>
-        <visual>
-            <origin rpy="0 0 1.57" xyz="0.1 0 -0.4"/>
-            <geometry>
-                <mesh filename="package://exotica_satellite_dynamics_solver/resources/robots/satellite/satellite_base2.dae" scale="1 1 1"/>
-            </geometry>
-        </visual>
+        <!-- <visual>
+            <origin rpy="0 0 0" xyz="0 0 0"/>
+            <geometry>
+                <mesh filename="package://exotica_satellite_dynamics_solver/resources/robots/satellite/satellite_base.dae" scale="1 1 1"/>
+            </geometry>
+        </visual> -->
         <xacro:if value="${show_outline == 1}">
             <visual>
@@ -285,4 +286,16 @@
         </inertial>
     </link>
+    <link name="heavy_object">
+        <visual>
+            <geometry>
+                <sphere radius="0.5"></sphere>
+            </geometry>
+        </visual>
+        <inertial>
+            <mass value="${heavy_object_mass}"></mass>
+            <origin rpy="0 0 0" xyz="0 0 1"/>
+            <inertia ixx="${heavy_object_mass * 0.5 * 0.5 * 2/5}" ixy="0.0" ixz="0.0" iyy="${heavy_object_mass * 0.5 * 0.5 * 2/5}" iyz="0.0" izz="${heavy_object_mass * 0.5 * 0.5 * 2/5}" />
+        </inertial>
+    </link>
     <joint name="base_to_arm" type="revolute">
         <parent link="base_link"/>
@@ -318,3 +331,8 @@
         <origin xyz="0 0 ${arm_segment_length + 0.1}"/>
     </joint>
+    <joint name="wrist_to_heavy_object" type="fixed">
+        <parent link="arm_end_eff"/>
+        <child link="heavy_object"/>
+        <origin xyz="0 0 0"/>
+    </joint>
 </robot>
