Commit message: Minor

File: resources/robots/satellite/satellite.urdf.xacro (robot description, xacro)
@@ -1,4 +1,5 @@
 <?xml version="1.0" encoding="utf-8"?>
-<robot name="satellite" xmlns:xacro="http://www.ros.org/wiki/xacro">
+<robot name="satellite"
+    xmlns:xacro="http://www.ros.org/wiki/xacro">
     <material name="blue">
         <color rgba="0 0 0.8 1"/>
@@ -25,11 +26,5 @@
             <mass value="${base_mass}"/>
             <origin xyz="0 0 0"/>
-            <inertia
-                ixx="${base_mass * 2.5 * 2.5 * 2/5}"
-                ixy="0.0" ixz="0.0"
-                iyy="${base_mass * 2.5 * 2.5 * 2/5}"
-                iyz="0.0"
-                izz="${base_mass * 4 * 4 * 2/5}"
-            />
+            <inertia ixx="${base_mass * 2.5 * 2.5 * 2/5}" ixy="0.0" ixz="0.0" iyy="${base_mass * 2.5 * 2.5 * 2/5}" iyz="0.0" izz="${base_mass * 4 * 4 * 2/5}" />
         </inertial>
         <!-- <visual>
@@ -217,13 +212,7 @@
         </visual>
         <inertial>
-            <mass value="0"/>
-            <origin xyz="0 0 0"/>
-            <inertia
-                ixx="0"
-                ixy="0.0" ixz="0.0"
-                iyy="0"
-                iyz="0.0"
-                izz="0"
-            />
+            <mass value="1e-12"/>
+            <origin xyz="0 0 0"/>
+            <inertia ixx="1e-12" ixy="0.0" ixz="0.0" iyy="1e-12" iyz="0.0" izz="1e-12"/>
         </inertial>
     </link>
@@ -239,11 +228,5 @@
             <mass value="${arm_segment_mass}"/>
             <origin xyz="0 0 0"/>
-            <inertia
-                ixx="${1/3 * arm_segment_mass * arm_segment_length * arm_segment_length}"
-                ixy="0.0" ixz="0.0"
-                iyy="0"
-                iyz="0.0"
-                izz="${1/3 * arm_segment_mass * arm_segment_length * arm_segment_length}"
-            />
+            <inertia ixx="${1/3 * arm_segment_mass * arm_segment_length * arm_segment_length}" ixy="0.0" ixz="0.0" iyy="0" iyz="0.0" izz="${1/3 * arm_segment_mass * arm_segment_length * arm_segment_length}" />
         </inertial>
     </link>
@@ -259,11 +242,5 @@
             <mass value="${arm_segment_mass}"/>
             <origin xyz="0 0 0"/>
-            <inertia
-                ixx="${1/3 * arm_segment_mass * arm_segment_length * arm_segment_length}"
-                ixy="0.0" ixz="0.0"
-                iyy="0"
-                iyz="0.0"
-                izz="${1/3 * arm_segment_mass * arm_segment_length * arm_segment_length}"
-            />
+            <inertia ixx="${1/3 * arm_segment_mass * arm_segment_length * arm_segment_length}" ixy="0.0" ixz="0.0" iyy="0" iyz="0.0" izz="${1/3 * arm_segment_mass * arm_segment_length * arm_segment_length}" />
         </inertial>
     </link>

Commit message: Fix inertia for arm

File: resources/robots/satellite/satellite.urdf.xacro (robot description, xacro)
@@ -19,5 +19,5 @@
     <xacro:property name="base_h" value="4" />
     <xacro:property name="arm_segment_length" value="2" />
-    <xacro:property name="arm_segment_mass" value="10" />
+    <xacro:property name="arm_segment_mass" value="1" />
     <!-- <link name="base_dummy"></link> -->
     <!-- links -->
@@ -66,5 +66,5 @@
         </inertial>
     </link>
-    <link name="left_array">
+    <!-- <link name="left_array">
         <visual>
             <geometry>
@@ -79,6 +79,6 @@
             <inertia ixx="1e-12" ixy="0.0" ixz="0.0" iyy="1e-12" iyz="0.0" izz="1e-12"/>
         </inertial>
-    </link>
-    <link name="right_array">
+    </link> -->
+    <!-- <link name="right_array">
         <visual>
             <geometry>
@@ -93,5 +93,5 @@
             <inertia ixx="1e-12" ixy="0.0" ixz="0.0" iyy="1e-12" iyz="0.0" izz="1e-12"/>
         </inertial>
-    </link>
+    </link> -->
     <link name="top_array">
         <visual>
@@ -182,5 +182,5 @@
         <origin xyz="0 0 2"/>
     </joint>
-    <joint name="base_to_left_array" type="fixed">
+    <!-- <joint name="base_to_left_array" type="fixed">
         <parent link="base_link"/>
         <child link="left_array"/>
@@ -191,5 +191,5 @@
         <child link="right_array"/>
         <origin xyz="1 -0.5 -1"/>
-    </joint>
+    </joint> -->
     <joint name="base_to_top_array" type="fixed">
         <parent link="base_link"/>
@@ -212,7 +212,7 @@
         </visual>
         <inertial>
-            <mass value="1e-12"/>
-            <origin xyz="0 0 0"/>
-            <inertia ixx="1e-12" ixy="0.0" ixz="0.0" iyy="1e-12" iyz="0.0" izz="1e-12"/>
+            <mass value="1e-3"/>
+            <origin xyz="0 0 0"/>
+            <inertia ixx="1e-3" ixy="0.0" ixz="0.0" iyy="1e-3" iyz="0.0" izz="1e-3"/>
         </inertial>
     </link>
@@ -227,6 +227,6 @@
         <inertial>
             <mass value="${arm_segment_mass}"/>
-            <origin xyz="0 0 0"/>
-            <inertia ixx="${1/3 * arm_segment_mass * arm_segment_length * arm_segment_length}" ixy="0.0" ixz="0.0" iyy="0" iyz="0.0" izz="${1/3 * arm_segment_mass * arm_segment_length * arm_segment_length}" />
+            <origin rpy="0 0 0" xyz="0 0 1"/>
+            <inertia ixx="${1/3 * arm_segment_mass * arm_segment_length * arm_segment_length}" ixy="0.0" ixz="0.0" iyy="1e-3" iyz="0.0" izz="${1/3 * arm_segment_mass * arm_segment_length * arm_segment_length}" />
         </inertial>
     </link>
@@ -241,6 +241,6 @@
         <inertial>
             <mass value="${arm_segment_mass}"/>
-            <origin xyz="0 0 0"/>
-            <inertia ixx="${1/3 * arm_segment_mass * arm_segment_length * arm_segment_length}" ixy="0.0" ixz="0.0" iyy="0" iyz="0.0" izz="${1/3 * arm_segment_mass * arm_segment_length * arm_segment_length}" />
+            <origin rpy="0 0 0" xyz="0 0 1"/>
+            <inertia ixx="${1/3 * arm_segment_mass * arm_segment_length * arm_segment_length}" ixy="0.0" ixz="0.0" iyy="1e-3" iyz="0.0" izz="${1/3 * arm_segment_mass * arm_segment_length * arm_segment_length}" />
         </inertial>
     </link>
@@ -248,5 +248,5 @@
         <parent link="base_link"/>
         <child link="arm_one"/>
-        <limit effort="100.0" lower="-1.57" upper="1.57" velocity="0.5"/>
+        <limit effort="1.0" lower="-1.57" upper="1.57" velocity="0.5"/>
         <axis xyz="1 0 0"/>
         <origin xyz="1.5 0 -0.25"/>
@@ -255,5 +255,5 @@
         <parent link="arm_one"/>
         <child link="arm_two"/>
-        <limit effort="100.0" lower="0" upper="3.14" velocity="0.5"/>
+        <limit effort="1.0" lower="0" upper="3.14" velocity="0.5"/>
         <axis xyz="0 1 0"/>
         <origin xyz="0 0 0"/>
@@ -262,5 +262,5 @@
         <parent link="arm_two"/>
         <child link="arm_three"/>
-        <limit effort="100.0" lower="-1.57" upper="1.57" velocity="0.5"/>
+        <limit effort="1.0" lower="-1.57" upper="1.57" velocity="0.5"/>
         <axis xyz="0 1 0"/>
         <origin xyz="0 0 2"/>

Commit message: Long Trajectory

File: resources/robots/satellite/satellite.urdf.xacro (robot description, xacro)
@@ -20,4 +20,5 @@
     <xacro:property name="arm_segment_length" value="2" />
     <xacro:property name="arm_segment_mass" value="1" />
+    <xacro:property name="show_outline" value="0" />
     <!-- <link name="base_dummy"></link> -->
     <!-- links -->
@@ -28,15 +29,17 @@
             <inertia ixx="${base_mass * 2.5 * 2.5 * 2/5}" ixy="0.0" ixz="0.0" iyy="${base_mass * 2.5 * 2.5 * 2/5}" iyz="0.0" izz="${base_mass * 4 * 4 * 2/5}" />
         </inertial>
-        <!-- <visual>
+        <visual>
             <origin rpy="0 0 0" xyz="0 0 0"/>
             <geometry>
                 <mesh filename="package://exotica_satellite_dynamics_solver/resources/robots/satellite/satellite_base.dae" scale="1 1 1"/>
             </geometry>
-        </visual> -->
-        <visual>
-            <geometry>
-                <box size="2.5 2.5 4"/>
-            </geometry>
-        </visual>
+        </visual>
+        <xacro:if value="${show_outline}">
+            <visual>
+                <geometry>
+                    <box size="2.5 2.5 4"/>
+                </geometry>
+            </visual>
+        </xacro:if>
         <!-- <collision>
             <origin rpy="0 0 0" xyz="0 0 0"/>
@@ -53,11 +56,13 @@
     <!-- antenna and communication arrays -->
     <link name="front">
-        <visual>
-            <geometry>
-                <cylinder length="4" radius="1"/>
-            </geometry>
-            <origin rpy="0 0 0" xyz="0 0 2"/>
-            <material name="black"/>
-        </visual>
+        <xacro:if value="${show_outline}">
+            <visual>
+                <geometry>
+                    <cylinder length="4" radius="1"/>
+                </geometry>
+                <origin rpy="0 0 0" xyz="0 0 2"/>
+                <material name="black"/>
+            </visual>
+        </xacro:if>
         <inertial>
             <mass value="1e-12"/>
@@ -95,11 +100,13 @@
     </link> -->
     <link name="top_array">
-        <visual>
-            <geometry>
-                <box size="2 4 0.2"/>
-            </geometry>
-            <origin rpy="0 0 0" xyz="0 2 0"/>
-            <material name="black"/>
-        </visual>
+        <xacro:if value="${show_outline}">
+            <visual>
+                <geometry>
+                    <box size="2 4 0.2"/>
+                </geometry>
+                <origin rpy="0 0 0" xyz="0 2 0"/>
+                <material name="black"/>
+            </visual>
+        </xacro:if>
         <inertial>
             <mass value="1e-12"/>
@@ -109,11 +116,13 @@
     </link>
     <link name="bot_array">
-        <visual>
-            <geometry>
-                <box size="2 4 0.2"/>
-            </geometry>
-            <origin rpy="0 0 0" xyz="0 -2 0"/>
-            <material name="black"/>
-        </visual>
+        <xacro:if value="${show_outline}">
+            <visual>
+                <geometry>
+                    <box size="2 4 0.2"/>
+                </geometry>
+                <origin rpy="0 0 0" xyz="0 -2 0"/>
+                <material name="black"/>
+            </visual>
+        </xacro:if>
         <inertial>
             <mass value="1e-12"/>
@@ -209,5 +218,5 @@
             </geometry>
             <origin rpy="0 0 0" xyz="0 0 0"/>
-            <material name="white"/>
+            <material name="green"/>
         </visual>
         <inertial>
@@ -223,5 +232,5 @@
             </geometry>
             <origin rpy="0 0 0" xyz="0 0 1"/>
-            <material name="white"/>
+            <material name="green"/>
         </visual>
         <inertial>
@@ -237,5 +246,5 @@
             </geometry>
             <origin rpy="0 0 0" xyz="0.2 0 -1"/>
-            <material name="white"/>
+            <material name="green"/>
         </visual>
         <inertial>

Commit message: Sparse ffdp examples

File: resources/robots/satellite/satellite.urdf.xacro (robot description, xacro)
@@ -14,5 +14,5 @@
         <color rgba="1 1 1 1"/>
     </material>
-    <xacro:property name="base_mass" value="60" />
+    <xacro:property name="base_mass" value="100" />
     <xacro:property name="base_w" value="2" />
     <xacro:property name="base_l" value="2" />
@@ -20,5 +20,5 @@
     <xacro:property name="arm_segment_length" value="2" />
     <xacro:property name="arm_segment_mass" value="1" />
-    <xacro:property name="show_outline" value="0" />
+    <xacro:property name="show_outline" value="1" />
     <!-- <link name="base_dummy"></link> -->
     <!-- links -->
@@ -29,11 +29,11 @@
             <inertia ixx="${base_mass * 2.5 * 2.5 * 2/5}" ixy="0.0" ixz="0.0" iyy="${base_mass * 2.5 * 2.5 * 2/5}" iyz="0.0" izz="${base_mass * 4 * 4 * 2/5}" />
         </inertial>
-        <visual>
+        <!-- <visual>
             <origin rpy="0 0 0" xyz="0 0 0"/>
             <geometry>
                 <mesh filename="package://exotica_satellite_dynamics_solver/resources/robots/satellite/satellite_base.dae" scale="1 1 1"/>
             </geometry>
-        </visual>
-        <xacro:if value="${show_outline}">
+        </visual> -->
+        <xacro:if value="${show_outline == 1}">
             <visual>
                 <geometry>
@@ -56,5 +56,5 @@
     <!-- antenna and communication arrays -->
     <link name="front">
-        <xacro:if value="${show_outline}">
+        <!-- <xacro:if value="${show_outline == 1}">
             <visual>
                 <geometry>
@@ -64,5 +64,5 @@
                 <material name="black"/>
             </visual>
-        </xacro:if>
+        </xacro:if> -->
         <inertial>
             <mass value="1e-12"/>
@@ -100,5 +100,5 @@
     </link> -->
     <link name="top_array">
-        <xacro:if value="${show_outline}">
+        <!-- <xacro:if value="${show_outline == 1}">
             <visual>
                 <geometry>
@@ -108,5 +108,5 @@
                 <material name="black"/>
             </visual>
-        </xacro:if>
+        </xacro:if> -->
         <inertial>
             <mass value="1e-12"/>
@@ -116,5 +116,5 @@
     </link>
     <link name="bot_array">
-        <xacro:if value="${show_outline}">
+        <!-- <xacro:if value="${show_outline == 1}">
             <visual>
                 <geometry>
@@ -124,5 +124,5 @@
                 <material name="black"/>
             </visual>
-        </xacro:if>
+        </xacro:if> -->
         <inertial>
             <mass value="1e-12"/>
@@ -259,5 +259,5 @@
         <limit effort="1.0" lower="-1.57" upper="1.57" velocity="0.5"/>
         <axis xyz="1 0 0"/>
-        <origin xyz="1.5 0 -0.25"/>
+        <origin xyz="1.25 0 -1"/>
     </joint>
     <joint name="arm_one_to_two" type="revolute">

Commit message: 2-stage point to target

File: resources/robots/satellite/satellite.urdf.xacro (robot description, xacro)
@@ -288,5 +288,5 @@
         <parent link="base_link"/>
         <child link="arm_base"/>
-        <limit effort="1.0" lower="-3.14" upper="3.14" velocity="0.5"/>
+        <limit effort="1.0" lower="-1.57" upper="1.57" velocity="0.5"/>
         <axis xyz="1 0 0"/>
         <origin xyz="1.25 0 -${arm_segment_length/2}"/>
@@ -295,5 +295,5 @@
         <parent link="arm_base"/>
         <child link="arm_shoulder"/>
-        <limit effort="1.0" lower="-3.14" upper="3.14" velocity="0.5"/>
+        <limit effort="1.0" lower="0" upper="1.57" velocity="0.5"/>
         <axis xyz="0 1 0"/>
         <origin xyz="0 0 0"/>
@@ -302,6 +302,6 @@
         <parent link="arm_shoulder"/>
         <child link="arm_elbow"/>
-        <limit effort="1.0" lower="-3.14" upper="3.14" velocity="0.5"/>
-        <axis xyz="0 1 0"/>
+        <limit effort="1.0" lower="0" upper="1.57" velocity="0.5"/>
+        <axis xyz="0 -1 0"/>
         <origin xyz="0 0 ${arm_segment_length}"/>
     </joint>
@@ -310,5 +310,5 @@
         <child link="arm_wrist"/>
         <limit effort="1.0" lower="-3.14" upper="3.14" velocity="0.5"/>
-        <axis xyz="1 0 0"/>
+        <axis xyz="-1 0 0"/>
         <origin xyz="0 0 -${arm_segment_length}"/>
     </joint>

Commit message: Better joint limits & combined example

File: resources/robots/satellite/satellite.urdf.xacro (robot description, xacro)
@@ -295,5 +295,5 @@
         <parent link="arm_base"/>
         <child link="arm_shoulder"/>
-        <limit effort="1.0" lower="0" upper="1.57" velocity="0.5"/>
+        <limit effort="1.0" lower="0" upper="3.14" velocity="0.5"/>
         <axis xyz="0 1 0"/>
         <origin xyz="0 0 0"/>
@@ -302,5 +302,5 @@
         <parent link="arm_shoulder"/>
         <child link="arm_elbow"/>
-        <limit effort="1.0" lower="0" upper="1.57" velocity="0.5"/>
+        <limit effort="1.0" lower="0" upper="3.14" velocity="0.5"/>
         <axis xyz="0 -1 0"/>
         <origin xyz="0 0 ${arm_segment_length}"/>
@@ -309,5 +309,5 @@
         <parent link="arm_elbow"/>
         <child link="arm_wrist"/>
-        <limit effort="1.0" lower="-3.14" upper="3.14" velocity="0.5"/>
+        <limit effort="1.0" lower="-300" upper="300" velocity="0.5"/>
         <axis xyz="-1 0 0"/>
         <origin xyz="0 0 -${arm_segment_length}"/>
