Commit message: Clean-up

File: resources/robots/satellite/satellite.urdf.xacro (robot description, xacro)
@@ -14,4 +14,7 @@
         <color rgba="0 1 0 1"/>
     </material>
+    <material name="red">
+        <color rgba="1 0 0 1"/>
+    </material>
     <material name="white">
         <color rgba="1 1 1 1"/>
@@ -21,8 +24,5 @@
     <xacro:property name="base_l" value="4" />
     <xacro:property name="base_h" value="11" />
-    <xacro:property name="arm_segment_length" value="3" />
-    <xacro:property name="arm_segment_mass" value="136" />
     <xacro:property name="show_outline" value="0" />
-    <!-- <link name="base_dummy"></link> -->
     <!-- links -->
     <link name="base_link">
@@ -33,7 +33,8 @@
         </inertial>
         <visual>
-            <origin rpy="0 0 1.57" xyz="0.1 0 -0.4"/>
+            <origin rpy="0 0 0" xyz="0 0 0"/>
             <geometry>
-                <mesh filename="package://exotica_satellite_dynamics_solver/resources/robots/satellite/satellite_base2.dae" scale="1 1 1"/>
+                <!-- <mesh filename="package://exotica_satellite_dynamics_solver/resources/robots/satellite/satellite_base.dae" scale="1 1 1"/> -->
+                <mesh filename="package://exotica_satellite_dynamics_solver/resources/robots/satellite/LORAL-1300MANIP.dae" />
             </geometry>
         </visual>
@@ -45,276 +46,56 @@
             </visual>
         </xacro:if>
-        <!-- <collision>
-            <origin rpy="0 0 0" xyz="0 0 0"/>
-            <geometry>
-                <mesh filename="package://exotica_satellite_dynamics_solver/resources/robots/quadrotor/quadrotor_base_convex_hull.stl"/>
-            </geometry>
-        </collision> -->
-    </link>
-    <!-- <joint name="base_to_dummy" type="fixed">
-        <parent link="base_dummy"/>
-        <child link="base_link"/>
-        <origin xyz="0 0 0"/>
-    </joint> -->
-    <!-- antenna and communication arrays -->
-    <link name="front">
-        <!-- <xacro:if value="${show_outline == 1}">
-            <visual>
-                <geometry>
-                    <cylinder length="4" radius="1"/>
-                </geometry>
-                <origin rpy="0 0 0" xyz="0 0 2"/>
-                <material name="black"/>
-            </visual>
-        </xacro:if> -->
-        <inertial>
-            <mass value="1e-12"/>
-            <origin xyz="0 0 0"/>
-            <inertia ixx="1e-12" ixy="0.0" ixz="0.0" iyy="1e-12" iyz="0.0" izz="1e-12"/>
-        </inertial>
-    </link>
-    <!-- <link name="left_array">
-        <visual>
-            <geometry>
-                <box size="12 0.2 2"/>
-            </geometry>
-            <origin rpy="0.785 0 0" xyz="-6 0 0"/>
-            <material name="white"/>
-        </visual>
-        <inertial>
-            <mass value="1e-12"/>
-            <origin xyz="0 0 0"/>
-            <inertia ixx="1e-12" ixy="0.0" ixz="0.0" iyy="1e-12" iyz="0.0" izz="1e-12"/>
-        </inertial>
-    </link> -->
-    <!-- <link name="right_array">
-        <visual>
-            <geometry>
-                <box size="12 0.2 2"/>
-            </geometry>
-            <origin rpy="0.785 0 0" xyz="6 0 0"/>
-            <material name="white"/>
-        </visual>
-        <inertial>
-            <mass value="1e-12"/>
-            <origin xyz="0 0 0"/>
-            <inertia ixx="1e-12" ixy="0.0" ixz="0.0" iyy="1e-12" iyz="0.0" izz="1e-12"/>
-        </inertial>
-    </link> -->
-    <link name="top_array">
-        <!-- <xacro:if value="${show_outline == 1}">
-            <visual>
-                <geometry>
-                    <box size="2 4 0.2"/>
-                </geometry>
-                <origin rpy="0 0 0" xyz="0 2 0"/>
-                <material name="black"/>
-            </visual>
-        </xacro:if> -->
-        <inertial>
-            <mass value="1e-12"/>
-            <origin xyz="0 0 0"/>
-            <inertia ixx="1e-12" ixy="0.0" ixz="0.0" iyy="1e-12" iyz="0.0" izz="1e-12"/>
-        </inertial>
-    </link>
-    <link name="bot_array">
-        <!-- <xacro:if value="${show_outline == 1}">
-            <visual>
-                <geometry>
-                    <box size="2 4 0.2"/>
-                </geometry>
-                <origin rpy="0 0 0" xyz="0 -2 0"/>
-                <material name="black"/>
-            </visual>
-        </xacro:if> -->
-        <inertial>
-            <mass value="1e-12"/>
-            <origin xyz="0 0 0"/>
-            <inertia ixx="1e-12" ixy="0.0" ixz="0.0" iyy="1e-12" iyz="0.0" izz="1e-12"/>
-        </inertial>
     </link>
     <!-- thrusters -->
-    <xacro:macro name="thruster" params="name origin">
+    <xacro:macro name="thruster" params="name xyz rpy">
         <link name="thruster_${name}">
             <visual>
                 <geometry>
-                    <box size="0.2 0.2 0.2"/>
+                    <box size="0.1 0.1 0.2"/>
                 </geometry>
                 <origin rpy="0 0 0" xyz="0 0 0"/>
                 <material name="green"/>
             </visual>
+            <visual>
+                <geometry>
+                    <box size="0.05 0.05 0.05"/>
+                </geometry>
+                <origin rpy="0 0 0" xyz="0 0 0.1"/>
+                <material name="red"/>
+            </visual>
             <inertial>
                 <mass value="0.001"/>
-                <!-- <origin xyz="0 0 0"/> -->
                 <inertia ixx="1e-3" ixy="0.0" ixz="0.0" iyy="1e-3" iyz="0.0" izz="1e-3"/>
             </inertial>
         </link>
-        <!-- Prismatic joints with no effort so pinocchio recognizes
-            them as controllable joints.
-         -->
         <joint name="base_to_thruster_${name}" type="fixed">
-            <!-- <limit effort="1e-10" lower="0" upper="1e-10" velocity="1e-10"/> -->
-            <!-- <axis xyz="${axis}"/> -->
-            <!-- <limit effort="1000.0" lower="0.0" upper="0.548" velocity="0.5"/> -->
             <parent link="base_link"/>
             <child link="thruster_${name}"/>
-            <origin xyz="${origin}"/>
+            <origin xyz="${xyz}" rpy="${rpy}"/>
         </joint>
     </xacro:macro>
-    <xacro:thruster name="bot" origin="0 0 -2"/>
-    <xacro:thruster name="bot_1" origin="0 -1.3 -1.8"/>
-    <xacro:thruster name="bot_2" origin="-1.3 0 -1.8"/>
-    <xacro:thruster name="bot_3" origin="0 1.3 -1.8"/>
-    <xacro:thruster name="bot_4" origin="1.3 0 -1.8"/>
-    <xacro:thruster name="top" origin="0 0 2"/>
-    <xacro:thruster name="top_1" origin="0 -1.3 1.8"/>
-    <xacro:thruster name="top_2" origin="-1.3 0 1.8"/>
-    <xacro:thruster name="top_3" origin="0 1.3 1.8"/>
-    <xacro:thruster name="top_4" origin="1.3 0 1.8"/>
-    <!-- <xacro:thruster name="bot_2" origin="-1.3 -1 -1.8"/> -->
-    <!-- <xacro:thruster name="bot_3" origin="1.3 -1 -1.8"/> -->
-    <!-- <xacro:thruster name="bot_4" origin="1 -1.3 -1.8"/> -->
-    <!-- <xacro:thruster name="bot_5" origin="1.3 1 -1.8"/> -->
-    <!-- <xacro:thruster name="bot_6" origin="1 1.3 -1.8"/> -->
-    <!-- <xacro:thruster name="bot_7" origin="-1 1.3 -1.8"/> -->
-    <!-- <xacro:thruster name="bot_8" origin="-1.3 1 -1.8"/> -->
-    <!-- <xacro:thruster name="top" origin="0 0 2"/> -->
-    <!-- <xacro:thruster name="top_1" origin="-1 -1.3 1.8"/> -->
-    <!-- <xacro:thruster name="top_2" origin="-1.3 -1 1.8"/> -->
-    <!-- <xacro:thruster name="top_3" origin="1.3 -1 1.8"/> -->
-    <!-- <xacro:thruster name="top_4" origin="1 -1.3 1.8"/> -->
-    <!-- <xacro:thruster name="top_5" origin="1.3 1 1.8"/> -->
-    <!-- <xacro:thruster name="top_6" origin="1 1.3 1.8"/> -->
-    <!-- <xacro:thruster name="top_7" origin="-1 1.3 1.8"/> -->
-    <!-- <xacro:thruster name="top_8" origin="-1.3 1 1.8"/> -->
-    <!-- joints -->
-    <joint name="base_to_front" type="fixed">
-        <parent link="base_link"/>
-        <child link="front"/>
-        <origin xyz="0 0 2"/>
-    </joint>
-    <!-- <joint name="base_to_left_array" type="fixed">
-        <parent link="base_link"/>
-        <child link="left_array"/>
-        <origin xyz="-1 -0.5 -1"/>
-    </joint>
-    <joint name="base_to_right_array" type="fixed">
-        <parent link="base_link"/>
-        <child link="right_array"/>
-        <origin xyz="1 -0.5 -1"/>
-    </joint> -->
-    <joint name="base_to_top_array" type="fixed">
-        <parent link="base_link"/>
-        <child link="top_array"/>
-        <origin xyz="0 1 -1"/>
-    </joint>
-    <joint name="base_to_bot_array" type="fixed">
-        <parent link="base_link"/>
-        <child link="bot_array"/>
-        <origin xyz="0 -1 -1"/>
-    </joint>
-    <!-- arm -->
-    <link name="arm_base">
-        <visual>
-            <geometry>
-                <cylinder length="0.5" radius="0.1"/>
-            </geometry>
-            <origin rpy="0 0 0" xyz="0 0 0"/>
-            <material name="green"/>
-        </visual>
-        <inertial>
-            <mass value="1e-3"/>
-            <origin xyz="0 0 0"/>
-            <inertia ixx="1e-3" ixy="0.0" ixz="0.0" iyy="1e-3" iyz="0.0" izz="1e-3"/>
-        </inertial>
-    </link>
-    <link name="arm_shoulder">
-        <visual>
-            <geometry>
-                <cylinder length="${arm_segment_length}" radius="0.1"/>
-            </geometry>
-            <origin rpy="0 0 0" xyz="0 0 ${arm_segment_length/2}"/>
-            <material name="green"/>
-        </visual>
-        <inertial>
-            <mass value="${arm_segment_mass}"/>
-            <origin rpy="0 0 0" xyz="0 0 1"/>
-            <inertia ixx="${1/3 * arm_segment_mass * arm_segment_length * arm_segment_length}" ixy="0.0" ixz="0.0" iyy="1e-3" iyz="0.0" izz="${1/3 * arm_segment_mass * arm_segment_length * arm_segment_length}" />
-        </inertial>
-    </link>
-    <link name="arm_elbow">
-        <visual>
-            <geometry>
-                <cylinder length="${arm_segment_length}" radius="0.1"/>
-            </geometry>
-            <origin rpy="0 0 0" xyz="0.1 0 -${arm_segment_length/2}"/>
-            <material name="green"/>
-        </visual>
-        <inertial>
-            <mass value="${arm_segment_mass}"/>
-            <origin rpy="0 0 0" xyz="0 0 1"/>
-            <inertia ixx="${1/3 * arm_segment_mass * arm_segment_length * arm_segment_length}" ixy="0.0" ixz="0.0" iyy="1e-3" iyz="0.0" izz="${1/3 * arm_segment_mass * arm_segment_length * arm_segment_length}" />
-        </inertial>
-    </link>
-    <link name="arm_wrist">
-        <visual>
-            <geometry>
-                <cylinder length="${arm_segment_length}" radius="0.1"/>
-            </geometry>
-            <origin rpy="0 0 0" xyz="0.2 0 ${arm_segment_length/2}"/>
-            <material name="green"/>
-        </visual>
-        <inertial>
-            <mass value="${arm_segment_mass}"/>
-            <origin rpy="0 0 0" xyz="0 0 1"/>
-            <inertia ixx="${1/3 * arm_segment_mass * arm_segment_length * arm_segment_length}" ixy="0.0" ixz="0.0" iyy="1e-3" iyz="0.0" izz="${1/3 * arm_segment_mass * arm_segment_length * arm_segment_length}" />
-        </inertial>
-    </link>
-    <link name="arm_end_eff">
-        <visual>
-            <geometry>
-                <cylinder length="0.2" radius="0.1"/>
-            </geometry>
-            <origin rpy="0 0 0" xyz="0.2 0 0"/>
-            <material name="yellow"/>
-        </visual>
-        <inertial>
-            <mass value="1e-5"/>
-            <origin rpy="0 0 0" xyz="0 0 1"/>
-            <inertia ixx="1e-3" ixy="0.0" ixz="0.0" iyy="1e-3" iyz="0.0" izz="1e-3" />
-        </inertial>
-    </link>
-    <joint name="base_to_arm" type="revolute">
-        <parent link="base_link"/>
-        <child link="arm_base"/>
-        <limit effort="1.0" lower="-1.57" upper="1.57" velocity="0.5"/>
-        <axis xyz="1 0 0"/>
-        <origin xyz="1.25 0 -${arm_segment_length/2}"/>
-    </joint>
-    <joint name="arm_base_to_shoulder" type="revolute">
-        <parent link="arm_base"/>
-        <child link="arm_shoulder"/>
-        <limit effort="1.0" lower="0" upper="3.14" velocity="0.5"/>
-        <axis xyz="0 1 0"/>
-        <origin xyz="0 0 0"/>
-    </joint>
-    <joint name="arm_shoulder_to_elbow" type="revolute">
-        <parent link="arm_shoulder"/>
-        <child link="arm_elbow"/>
-        <limit effort="1.0" lower="0" upper="3.14" velocity="0.5"/>
-        <axis xyz="0 -1 0"/>
-        <origin xyz="0 0 ${arm_segment_length}"/>
-    </joint>
-    <joint name="arm_elbow_to_wrist" type="revolute">
-        <parent link="arm_elbow"/>
-        <child link="arm_wrist"/>
-        <limit effort="1.0" lower="-300" upper="300" velocity="0.5"/>
-        <axis xyz="-1 0 0"/>
-        <origin xyz="0 0 -${arm_segment_length}"/>
-    </joint>
-    <joint name="arm_wrist_to_end_eff" type="fixed">
-        <parent link="arm_wrist"/>
-        <child link="arm_end_eff"/>
-        <origin xyz="0 0 ${arm_segment_length + 0.1}"/>
-    </joint>
+    <!-- Main thruster -->
+    <xacro:thruster name="bot_0" xyz="0 0 -2.4" rpy="0 -3.1415 0"/>
+    <!-- Steering thrusters -->
+    <xacro:thruster name="bot_1" xyz="1.0 -1.2 -2" rpy="1.57 0 1.57"/>
+    <xacro:thruster name="bot_2" xyz="-1.0 1.2 -2" rpy="0 -1.57 0"/>
+    <xacro:thruster name="bot_3" xyz="0.9 1.4 -2" rpy="-1.57 0 0"/>
+    <xacro:thruster name="bot_4" xyz="-0.9 -1.4 -2" rpy="1.57 0 0"/>
+    <!-- More steering thrusters -->
+    <xacro:thruster name="bot_5" xyz="0.9 -1.4 -2" rpy="1.57 0 0"/>
+    <xacro:thruster name="bot_6" xyz="-0.9 1.4 -2" rpy="-1.57 0 0"/>
+    <xacro:thruster name="bot_7" xyz="1.0 1.2 -2" rpy="0 1.57 0"/>
+    <xacro:thruster name="bot_8" xyz="-1.0 -1.2 -2" rpy="0 -1.57 0"/>
+    <!-- Main thruster -->
+    <xacro:thruster name="top_0" xyz="0 0 1.7" rpy="0 0 0"/>
+    <!-- Steering thrusters -->
+    <xacro:thruster name="top_1" xyz="1.0 -1.2 1.5" rpy="1.57 0 1.57"/>
+    <xacro:thruster name="top_2" xyz="-1.0 1.2 1.5" rpy="0 -1.57 0"/>
+    <xacro:thruster name="top_3" xyz="0.9 1.4 1.5" rpy="-1.57 0 0"/>
+    <xacro:thruster name="top_4" xyz="-0.9 -1.4 1.5" rpy="1.57 0 0"/>
+    <!-- More steering thrusters -->
+    <xacro:thruster name="top_5" xyz="0.9 -1.4 1.5" rpy="1.57 0 0"/>
+    <xacro:thruster name="top_6" xyz="-0.9 1.4 1.5" rpy="-1.57 0 0"/>
+    <xacro:thruster name="top_7" xyz="1.0 1.2 1.5" rpy="0 1.57 0"/>
+    <xacro:thruster name="top_8" xyz="-1.0 -1.2 1.5" rpy="0 -1.57 0"/>
 </robot>
